Commit message: fix some issues

File: limo_challenges/urdf/marker.xacro (robot description, xacro)
@@ -1,9 +1,10 @@
 <?xml version="1.0"?>
 <robot xmlns:xacro="http://www.ros.org/wiki/xacro">
-    <xacro:property name="num_marker" value="0" />
+    <xacro:arg name="marker" default="0" />
+    <xacro:property name="NumMarker" value="$(arg marker)" />
     <xacro:property name="dim" value="0.3" />
     <xacro:property name="m" value="100" />
-<!--  <xacro:macro name="aruco_cube" params="num_marker dim m ">  -->
-<link name="marker">
+<!--  <xacro:macro name="aruco_cube" params="marker dim m ">  -->
+<link name="marker${NumMarker}">
    <inertial>
       <origin xyz="0 0 0" />
@@ -12,11 +13,13 @@
     </inertial>
     <visual>
+        <origin xyz="0 0 ${0.25*dim}" />
       <geometry>
-        <mesh filename="package://limo_challenges/urdf/marker${num_marker}/meshes/Marker${num_marker}.dae" scale="${2.0*dim} ${2.0*dim} ${2.0*dim}"/>
+        <mesh filename="package://limo_challenges/urdf/marker${NumMarker}/meshes/Marker${NumMarker}.dae" scale="${2.0*dim} ${2.0*dim} ${2.0*dim}"/>
       </geometry>
     </visual>
     <collision>
+    <origin xyz="0 0 ${0.5*dim}" />
       <geometry>
-        <box size="${dim} ${dim*0.1} ${dim*1.2}" />
+        <box size="${0.1*dim} ${dim} ${1.5*dim}" />
       </geometry>
     </collision>

File: limo_challenges/urdf/obstacle.xacro (robot description, xacro)
@@ -13,10 +13,10 @@
     <visual>
       <geometry>
-        <box size="${dim} ${dim*0.1} ${dim*0.1}" />
+        <box size="${dim} ${dim*0.1} ${dim*0.15}" />
       </geometry>
     </visual>
     <collision>
       <geometry>
-        <box size="${dim} ${dim*0.1} ${dim*0.1}" />
+        <box size="${dim} ${dim*0.1} ${dim*0.15}" />
       </geometry>
     </collision>
